File: kicad/solder.kicad_pcb (KiCad board)
At the start: 2 copper layers, 59.3 x 65.7 mm, 11 parts, among them SW1 SW_Push, SW3 SW_Push, SW5 SW_Push

Commit message: update pcb
Changed lines of the file:
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@@
 		(tags "LED")
 		(property "Reference" "D1"
-			(at 1.27 -3.96 360)
+			(at 1.27 -3.96 0)
 			(layer "F.SilkS")
 			(effects
@@
 		)
 		(property "Value" "LED"
-			(at 1.27 3.96 360)
+			(at 1.27 3.96 0)
 			(layer "F.Fab")
 			(effects
@@
 		)
 		(property "Footprint" ""
-			(at 0 0 360)
+			(at 0 0 180)
 			(layer "F.Fab")
 			(hide yes)
@@
 		)
 		(property "Datasheet" ""
-			(at 0 0 360)
+			(at 0 0 0)
 			(layer "F.Fab")
 			(hide yes)
@@
 		)
 		(property "Description" "Light emitting diode"
-			(at 0 0 360)
+			(at 0 0 0)
 			(layer "F.Fab")
 			(hide yes)
@@
 		)
 		(fp_text user "${REFERENCE}"
-			(at 1.27 0 360)
+			(at 1.27 0 0)
 			(layer "F.Fab")
 			(effects
@@
 		(tags "Keystone type 3034 coin cell retainer")
 		(property "Reference" "BT1"
-			(at 0 11.5 360)
+			(at 0 11.5 0)
 			(layer "B.SilkS")
 			(effects
@@
 		)
 		(property "Value" "Battery_Cell"
-			(at 0 -11.5 360)
+			(at 0 -11.5 0)
 			(layer "B.Fab")
 			(effects
@@
 		)
 		(property "Footprint" ""
-			(at 0 0 360)
-			(layer "B.Fab")
+			(at 0 0 0)
+			(layer "F.Fab")
 			(hide yes)
 			(effects
@@
 					(thickness 0.15)
 				)
-				(justify mirror)
 			)
 		)
@@
 		)
 		(property "Footprint" ""
-			(at 0 0 0)
-			(layer "B.Fab")
+			(at 0 0 180)
+			(layer "F.Fab")
 			(hide yes)
 			(effects
@@
 					(thickness 0.15)
 				)
-				(justify mirror)
 			)
 		)
@@
 		(tags "tact sw push 6mm")
 		(property "Reference" "SW3"
-			(at 3.25 2 360)
+			(at 3.25 2 0)
 			(layer "B.SilkS")
 			(effects
@@
 			)
 		)
-		(property "Footprint" ""
-			(at 0 0 360)
+		(property "Value" "SW_Push"
+			(at 3.75 -6.7 0)
 			(layer "B.Fab")
-			(hide yes)
 			(effects
 				(font
-					(size 1.27 1.27)
+					(size 1 1)
 					(thickness 0.15)
 				)
@@
 			)
 		)
-		(property "Datasheet" ""
-			(at 0 0 180)
-			(unlocked yes)
-			(layer "B.Fab")
+		(property "Footprint" ""
+			(at 0 0 0)
+			(layer "F.Fab")
 			(hide yes)
 			(effects
@@
 					(thickness 0.15)
 				)
-				(justify mirror)
 			)
 		)
-		(property "Description" "Push button switch, generic, two pins"
+		(property "Datasheet" ""
 			(at 0 0 180)
 			(unlocked yes)
@@
 			)
 		)
-		(property "Value" "SW_Push"
-			(at 3.75 -6.7 360)
+		(property "Description" "Push button switch, generic, two pins"
+			(at 0 0 180)
+			(unlocked yes)
 			(layer "B.Fab")
+			(hide yes)
 			(effects
 				(font
-					(size 1 1)
+					(size 1.27 1.27)
 					(thickness 0.15)
 				)
@@
 		)
 		(fp_text user "${REFERENCE}"
-			(at 3.25 -2.25 360)
+			(at 3.25 -2.25 0)
 			(layer "B.Fab")
 			(effects
@@
 		(property "Footprint" ""
 			(at 0 0 90)
-			(layer "B.Fab")
+			(layer "F.Fab")
 			(hide yes)
 			(effects
@@
 					(thickness 0.15)
 				)
-				(justify mirror)
 			)
 		)
@@
 		(property "Footprint" ""
 			(at 0 0 90)
-			(layer "B.Fab")
+			(layer "F.Fab")
 			(hide yes)
 			(effects
@@
 					(thickness 0.15)
 				)
-				(justify mirror)
 			)
 		)
@@
 			)
 		)
-		(property "Footprint" ""
-			(at 0 0 90)
+		(property "Value" "SW_Push"
+			(at 3.75 -6.7 90)
 			(layer "B.Fab")
-			(hide yes)
 			(effects
 				(font
-					(size 1.27 1.27)
+					(size 1 1)
 					(thickness 0.15)
 				)
@@
 			)
 		)
-		(property "Datasheet" ""
-			(at 0 0 -90)
-			(unlocked yes)
-			(layer "B.Fab")
+		(property "Footprint" ""
+			(at 0 0 90)
+			(layer "F.Fab")
 			(hide yes)
 			(effects
@@
 					(thickness 0.15)
 				)
-				(justify mirror)
 			)
 		)
-		(property "Description" "Push button switch, generic, two pins"
+		(property "Datasheet" ""
 			(at 0 0 -90)
 			(unlocked yes)
@@
 			)
 		)
-		(property "Value" "SW_Push"
-			(at 3.75 -6.7 90)
+		(property "Description" "Push button switch, generic, two pins"
+			(at 0 0 -90)
+			(unlocked yes)
 			(layer "B.Fab")
+			(hide yes)
 			(effects
 				(font
-					(size 1 1)
+					(size 1.27 1.27)
 					(thickness 0.15)
 				)
@@
 		(tags "Resistor Axial_DIN0207 series Axial Horizontal pin pitch 7.62mm 0.25W = 1/4W length 6.3mm diameter 2.5mm")
 		(property "Reference" "R1"
-			(at 3.81 2.37 360)
+			(at 3.81 2.37 0)
 			(layer "B.SilkS")
 			(effects
@@
 		)
 		(property "Value" "R"
-			(at 3.81 -2.37 360)
+			(at 3.81 -2.37 0)
 			(layer "B.Fab")
 			(effects
@@
 		)
 		(property "Footprint" ""
-			(at 0 0 360)
-			(layer "B.Fab")
+			(at 0 0 0)
+			(layer "F.Fab")
 			(hide yes)
 			(effects
@@
 					(thickness 0.15)
 				)
-				(justify mirror)
 			)
 		)
@@
 		)
 		(fp_text user "${REFERENCE}"
-			(at 3.81 0 360)
+			(at 3.81 0 0)
 			(layer "B.Fab")
 			(effects
@@
 		)
 		(stroke
-			(width 0)
+			(width 0.1)
 			(type solid)
 		)

Commit message: new changes
Parts:
- added G***: LOGO, LOGO, B.Cu at (215.0, 62.0)
- added G***: LOGO, LOGO, B.Cu at (182.0, 74.5)
- added G***: LOGO, LOGO, B.Cu at (216.0, 105.5)
